File: rp2350-dev-board.kicad_pcb (KiCad board)
At the start: 2 copper layers, 48 parts, among them J1 USB4105-GF-A, J2 Conn_02x20_Odd_Even, J3 Conn_02x20_Odd_Even, SW1 RST, SW2 BOOTSEL, U1 W25Q128JVS, U2 RP2350B, U3 TPS6285021HQDRLRQ1, Y1 ABM8-272-T3 12MHz/10pF

Commit message: wip
Parts:
- C1, C10, C11, C12, C13, C14, C15, C16, C17, C18, C19, C2, C20, C21, C22, C23, C24, C25, C26, C27, C4, C5, C6, C7: footprint Resistor_SMD:R_0402_1005Metric_Pad0.72x0.64mm_HandSolder -> Capacitor_SMD:C_0402_1005Metric_Pad0.74x0.62mm_HandSolder
- R1, R2, R3, R4: footprint Resistor_SMD:R_0805_2012Metric_Pad1.20x1.40mm_HandSolder -> Resistor_SMD:R_0402_1005Metric_Pad0.72x0.64mm_HandSolder
- moved C1 555.1 mm to (146.7, 55.8)
- moved C10 555.1 mm to (146.7, 67.9)
- moved C11 555.1 mm to (141.9, 67.9)
- moved C12 555.1 mm to (146.7, 70.9)
- moved C13 555.1 mm to (151.5, 64.8)
- moved C14 555.1 mm to (137.1, 55.8)
- moved C15 555.1 mm to (137.1, 67.9)
- moved C16 555.1 mm to (137.1, 58.8)
- moved C17 555.1 mm to (137.1, 70.9)
- moved C18 555.1 mm to (146.7, 58.8)
- moved C19 555.1 mm to (137.1, 61.8)
- moved C2 555.1 mm to (141.9, 73.9)
- moved C20 555.1 mm to (137.1, 73.9)
- moved C21 555.1 mm to (137.1, 64.8)
- moved C22 555.1 mm to (141.9, 55.8)
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
Commit message: initial layout
Parts:
- added U4: LM66100DCK, Package_TO_SOT_SMD:SOT-363_SC-70-6, F.Cu at (134.4, 123.8)
- J2: value Conn_02x20_Odd_Even -> EXT1
- J3: value Conn_02x20_Odd_Even -> EXT2
- moved C9 108.4 mm to (134.1, 162.8)
- moved C4 107.6 mm to (117.9, 164.1)
- moved C3 107.4 mm to (117.6, 160.8)
- moved C23 91.2 mm to (136.1, 149.9)
- moved C19 89.6 mm to (134.1, 151.4)
- moved C26 87.9 mm to (125.7, 151.9)
- moved U3 87.4 mm to (122.2, 161.3)
- moved C8 86.8 mm to (133.9, 159.8)
- moved C5 84.8 mm to (139.7, 146.3)
- moved R4 84.4 mm to (138.6, 148.8)
- moved R8 83.6 mm to (146.5, 150.0)
- moved C11 82.9 mm to (141.6, 150.8)
- moved C22 82.8 mm to (124.0, 136.7)
- moved C15 82.1 mm to (121.9, 148.6)
- moved C7 81.8 mm to (142.7, 146.6)
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Connections:
- J1 pad A4: +5V -> Net-(U4-VIN)
- J1 pad A9: +5V -> Net-(U4-VIN)
- J1 pad B4: +5V -> Net-(U4-VIN)
- J1 pad B9: +5V -> Net-(U4-VIN)
- J2 pad 1: /GPIO0 -> unconnected-(J2-Pin_1-Pad1)
- J2 pad 10: /GPIO24 -> unconnected-(J2-Pin_10-Pad10)
- J2 pad 11: /GPIO5 -> unconnected-(J2-Pin_11-Pad11)
- J2 pad 12: /GPIO25 -> unconnected-(J2-Pin_12-Pad12)
- J2 pad 13: /GPIO6 -> unconnected-(J2-Pin_13-Pad13)
- J2 pad 14: /GPIO26 -> unconnected-(J2-Pin_14-Pad14)
- J2 pad 15: /GPIO7 -> /GPIO4
- J2 pad 16: /GPIO27 -> unconnected-(J2-Pin_16-Pad16)
- J2 pad 17: /GPIO8 -> /GPIO6
- J2 pad 18: /GPIO28 -> /GPIO5
- J2 pad 19: /GPIO9 -> /GPIO8
- J2 pad 2: /GPIO20 -> unconnected-(J2-Pin_2-Pad2)
- J2 pad 20: /GPIO29 -> /GPIO7
- J2 pad 21: /GPIO10 -> unconnected-(J2-Pin_21-Pad21)
- J2 pad 22: /GPIO30 -> unconnected-(J2-Pin_22-Pad22)
- J2 pad 23: /GPIO11 -> unconnected-(J2-Pin_23-Pad23)
- J2 pad 24: /GPIO31 -> unconnected-(J2-Pin_24-Pad24)
- J2 pad 25: /GPIO12 -> /GPIO10
- J2 pad 26: /GPIO32 -> /GPIO9
- J2 pad 27: /GPIO13 -> /GPIO12
- J2 pad 28: /GPIO33 -> /GPIO11
- J2 pad 3: /GPIO1 -> unconnected-(J2-Pin_3-Pad3)
- J2 pad 30: /GPIO34 -> /GPIO13
- J2 pad 31: /GPIO15 -> /GPIO16
- J2 pad 32: /GPIO35 -> /GPIO15
- J2 pad 33: /GPIO16 -> /GPIO18
- J2 pad 34: /GPIO36 -> /GPIO17
- J2 pad 35: /GPIO17 -> /GPIO20
- J2 pad 36: /GPIO37 -> /GPIO19
- J2 pad 37: /GPIO18 -> unconnected-(J2-Pin_37-Pad37)
- J2 pad 38: /GPIO38 -> unconnected-(J2-Pin_38-Pad38)
- J2 pad 39: /GPIO19 -> unconnected-(J2-Pin_39-Pad39)
- J2 pad 4: /GPIO21 -> unconnected-(J2-Pin_4-Pad4)
- J2 pad 40: /GPIO39 -> unconnected-(J2-Pin_40-Pad40)
- J2 pad 5: /GPIO2 -> unconnected-(J2-Pin_5-Pad5)
- J2 pad 6: /GPIO22 -> unconnected-(J2-Pin_6-Pad6)
- J2 pad 7: /GPIO3 -> unconnected-(J2-Pin_7-Pad7)
- J2 pad 8: /GPIO23 -> unconnected-(J2-Pin_8-Pad8)
- J2 pad 9: /GPIO4 -> unconnected-(J2-Pin_9-Pad9)
- J3 pad 1: /SWCLK -> unconnected-(J3-Pin_1-Pad1)
- J3 pad 10: unconnected-(J3-Pin_10-Pad10) -> /GPIO43
- J3 pad 12: unconnected-(J3-Pin_12-Pad12) -> /GPIO41
- J3 pad 13: /GPIO43 -> /GPIO40
- J3 pad 14: unconnected-(J3-Pin_14-Pad14) -> /GPIO39
- J3 pad 15: /GPIO44 -> /GPIO38
- J3 pad 16: unconnected-(J3-Pin_16-Pad16) -> /GPIO37
- J3 pad 17: /GPIO45 -> /GPIO36
- J3 pad 18: unconnected-(J3-Pin_18-Pad18) -> /GPIO35
- J3 pad 19: /GPIO46 -> /GPIO34
- J3 pad 20: unconnected-(J3-Pin_20-Pad20) -> /GPIO33
- J3 pad 21: /GPIO47 -> /GPIO32
- J3 pad 22: unconnected-(J3-Pin_22-Pad22) -> /GPIO31
- J3 pad 23: /BOOTSEL# -> /GPIO30
- J3 pad 24: unconnected-(J3-Pin_24-Pad24) -> /GPIO29
- J3 pad 25: unconnected-(J3-Pin_25-Pad25) -> /GPIO28
- J3 pad 26: unconnected-(J3-Pin_26-Pad26) -> /RUN
- J3 pad 27: unconnected-(J3-Pin_27-Pad27) -> /SWCLK
- J3 pad 29: unconnected-(J3-Pin_29-Pad29) -> /SWDIO
- J3 pad 3: /SWDIO -> unconnected-(J3-Pin_3-Pad3)
- J3 pad 30: unconnected-(J3-Pin_30-Pad30) -> /GPIO27
- J3 pad 31: unconnected-(J3-Pin_31-Pad31) -> /GPIO26
- J3 pad 32: unconnected-(J3-Pin_32-Pad32) -> /GPIO25
- J3 pad 33: unconnected-(J3-Pin_33-Pad33) -> /GPIO24
- J3 pad 34: unconnected-(J3-Pin_34-Pad34) -> /GPIO23
- J3 pad 35: unconnected-(J3-Pin_35-Pad35) -> /GPIO22
- J3 pad 36: unconnected-(J3-Pin_36-Pad36) -> /GPIO21
- J3 pad 5: /RUN -> unconnected-(J3-Pin_5-Pad5)
- J3 pad 6: unconnected-(J3-Pin_6-Pad6) -> /GPIO47
- J3 pad 7: /GPIO40 -> /GPIO46
- J3 pad 8: unconnected-(J3-Pin_8-Pad8) -> /GPIO45
- J3 pad 9: /GPIO41 -> /GPIO44
Routing:
- added copper zone on B.Cu, net GND
- added copper zone on F.Cu, net GND

Commit message: wip
Parts:
- added C28: 100nF, Capacitor_SMD:C_0402_1005Metric_Pad0.74x0.62mm_HandSolder, B.Cu at (118.4, 131.6)
- added D2: GREEN 2.1V 20mA, LED_SMD:LED_0805_2012Metric_Pad1.15x1.40mm_HandSolder, F.Cu at (145.8, 129.0)
- added R10: 1K, Resistor_SMD:R_0805_2012Metric_Pad1.20x1.40mm_HandSolder, F.Cu at (141.5, 129.3)
- added R11: 10K, Resistor_SMD:R_0805_2012Metric_Pad1.20x1.40mm_HandSolder, B.Cu at (125.7, 125.5)
- added U5: APS6404L-3SQRx-SN, Package_SO:SOIC-8_3.9x4.9mm_P1.27mm, B.Cu at (118.6, 127.5)
- moved C4 28.6 mm to (128.7, 137.7)
- moved C3 28.2 mm to (128.0, 134.6)
- moved U3 27.7 mm to (131.8, 135.4)
- moved L2 26.1 mm to (135.4, 135.1)
- moved C8 26.0 mm to (139.4, 134.4)
- moved C9 26.0 mm to (139.4, 137.4)
- moved C27 9.11 mm to (127.8, 142.2)
- moved C20 8.61 mm to (120.5, 146.6)
- moved C13 8.61 mm to (142.4, 152.7)
- moved C14 8.61 mm to (132.5, 143.6)
- moved C16 8.61 mm to (135.5, 145.9)
- moved C18 8.61 mm to (129.9, 143.6)
- moved C19 8.61 mm to (132.5, 159.8)
- moved C22 8.61 mm to (122.3, 145.1)
- moved C6 8.61 mm to (137.2, 159.2)
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
Commit message: add gnd and power to headers
Connections:
- J2 pad 1: unconnected-(J2-Pin_1-Pad1) -> GND
- J2 pad 10: unconnected-(J2-Pin_10-Pad10) -> /GPIO3
- J2 pad 11: unconnected-(J2-Pin_11-Pad11) -> /GPIO0
- J2 pad 12: unconnected-(J2-Pin_12-Pad12) -> /GPIO1
- J2 pad 2: unconnected-(J2-Pin_2-Pad2) -> GND
- J2 pad 21: unconnected-(J2-Pin_21-Pad21) -> +3.3V
- J2 pad 22: unconnected-(J2-Pin_22-Pad22) -> +3.3V
- J2 pad 23: unconnected-(J2-Pin_23-Pad23) -> GND
- J2 pad 24: unconnected-(J2-Pin_24-Pad24) -> GND
- J2 pad 3: unconnected-(J2-Pin_3-Pad3) -> +3.3V
- J2 pad 37: unconnected-(J2-Pin_37-Pad37) -> +3.3V
- J2 pad 38: unconnected-(J2-Pin_38-Pad38) -> +3.3V
- J2 pad 39: unconnected-(J2-Pin_39-Pad39) -> GND
- J2 pad 4: unconnected-(J2-Pin_4-Pad4) -> +3.3V
- J2 pad 40: unconnected-(J2-Pin_40-Pad40) -> GND
- J2 pad 5: unconnected-(J2-Pin_5-Pad5) -> +5V
- J2 pad 6: unconnected-(J2-Pin_6-Pad6) -> /BOOTSEL#
- J2 pad 7: unconnected-(J2-Pin_7-Pad7) -> +5V
- J2 pad 9: unconnected-(J2-Pin_9-Pad9) -> /GPIO2
- J3 pad 1: unconnected-(J3-Pin_1-Pad1) -> +3.3V
- J3 pad 2: unconnected-(J3-Pin_2-Pad2) -> GND
- J3 pad 28: unconnected-(J3-Pin_28-Pad28) -> GND
- J3 pad 3: unconnected-(J3-Pin_3-Pad3) -> GND
- J3 pad 37: unconnected-(J3-Pin_37-Pad37) -> +3.3V
- J3 pad 38: unconnected-(J3-Pin_38-Pad38) -> GND
- J3 pad 39: unconnected-(J3-Pin_39-Pad39) -> GND
- J3 pad 4: unconnected-(J3-Pin_4-Pad4) -> +3.3V
- J3 pad 40: unconnected-(J3-Pin_40-Pad40) -> +3.3V
- J3 pad 5: unconnected-(J3-Pin_5-Pad5) -> GND
Changed lines of the file:
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@@
 			(layers "*.Cu" "*.Mask")
 			(remove_unused_layers no)
-			(net "unconnected-(J3-Pin_1-Pad1)")
+			(net "+3.3V")
 			(pinfunction "Pin_1_1")
 			(pintype "passive")
@@
 			(layers "*.Cu" "*.Mask")
 			(remove_unused_layers no)
-			(net "unconnected-(J3-Pin_2-Pad2)")
+			(net "GND")
 			(pinfunction "Pin_2_2")
 			(pintype "passive")
@@
 			(layers "*.Cu" "*.Mask")
 			(remove_unused_layers no)
-			(net "unconnected-(J3-Pin_3-Pad3)")
+			(net "GND")
 			(pinfunction "Pin_3_3")
 			(pintype "passive")
@@
 			(layers "*.Cu" "*.Mask")
 			(remove_unused_layers no)
-			(net "unconnected-(J3-Pin_4-Pad4)")
+			(net "+3.3V")
 			(pinfunction "Pin_4_4")
 			(pintype "passive")
@@
 			(layers "*.Cu" "*.Mask")
 			(remove_unused_layers no)
-			(net "unconnected-(J3-Pin_5-Pad5)")
+			(net "GND")
 			(pinfunction "Pin_5_5")
 			(pintype "passive")
@@
 			(layers "*.Cu" "*.Mask")
 			(remove_unused_layers no)
-			(net "unconnected-(J3-Pin_28-Pad28)")
+			(net "GND")
 			(pinfunction "Pin_28_28")
 			(pintype "passive")
@@
 			(layers "*.Cu" "*.Mask")
 			(remove_unused_layers no)
-			(net "unconnected-(J3-Pin_37-Pad37)")
+			(net "+3.3V")
 			(pinfunction "Pin_37_37")
 			(pintype "passive")
@@
 			(layers "*.Cu" "*.Mask")
 			(remove_unused_layers no)
-			(net "unconnected-(J3-Pin_38-Pad38)")
+			(net "GND")
 			(pinfunction "Pin_38_38")
 			(pintype "passive")
@@
 			(layers "*.Cu" "*.Mask")
 			(remove_unused_layers no)
-			(net "unconnected-(J3-Pin_39-Pad39)")
+			(net "GND")
 			(pinfunction "Pin_39_39")
 			(pintype "passive")
@@
 			(layers "*.Cu" "*.Mask")
 			(remove_unused_layers no)
-			(net "unconnected-(J3-Pin_40-Pad40)")
+			(net "+3.3V")
 			(pinfunction "Pin_40_40")
 			(pintype "passive")
@@
 			(layers "*.Cu" "*.Mask")
 			(remove_unused_layers no)
-			(net "unconnected-(J2-Pin_1-Pad1)")
+			(net "GND")
 			(pinfunction "Pin_1_1")
 			(pintype "passive")
@@
 			(layers "*.Cu" "*.Mask")
 			(remove_unused_layers no)
-			(net "unconnected-(J2-Pin_2-Pad2)")
+			(net "GND")
 			(pinfunction "Pin_2_2")
 			(pintype "passive")
@@
 			(layers "*.Cu" "*.Mask")
 			(remove_unused_layers no)
-			(net "unconnected-(J2-Pin_3-Pad3)")
+			(net "+3.3V")
 			(pinfunction "Pin_3_3")
 			(pintype "passive")
@@
 			(layers "*.Cu" "*.Mask")
 			(remove_unused_layers no)
-			(net "unconnected-(J2-Pin_4-Pad4)")
+			(net "+3.3V")
 			(pinfunction "Pin_4_4")
 			(pintype "passive")
@@
 			(layers "*.Cu" "*.Mask")
 			(remove_unused_layers no)
-			(net "unconnected-(J2-Pin_5-Pad5)")
+			(net "+5V")
 			(pinfunction "Pin_5_5")
 			(pintype "passive")
@@
 			(layers "*.Cu" "*.Mask")
 			(remove_unused_layers no)
-			(net "unconnected-(J2-Pin_6-Pad6)")
+			(net "/BOOTSEL#")
 			(pinfunction "Pin_6_6")
 			(pintype "passive")
@@
 			(layers "*.Cu" "*.Mask")
 			(remove_unused_layers no)
-			(net "unconnected-(J2-Pin_7-Pad7)")
+			(net "+5V")
 			(pinfunction "Pin_7_7")
 			(pintype "passive")
@@
 			(net "unconnected-(J2-Pin_8-Pad8)")
 			(pinfunction "Pin_8_8")
-			(pintype "passive")
+			(pintype "passive+no_connect")
 		)
 		(pad "9" thru_hole circle
@@
 			(layers "*.Cu" "*.Mask")
 			(remove_unused_layers no)
-			(net "unconnected-(J2-Pin_9-Pad9)")
+			(net "/GPIO2")
 			(pinfunction "Pin_9_9")
 			(pintype "passive")
@@
 			(layers "*.Cu" "*.Mask")
 			(remove_unused_layers no)
-			(net "unconnected-(J2-Pin_10-Pad10)")
+			(net "/GPIO3")
 			(pinfunction "Pin_10_10")
 			(pintype "passive")
@@
 			(layers "*.Cu" "*.Mask")
 			(remove_unused_layers no)
-			(net "unconnected-(J2-Pin_11-Pad11)")
+			(net "/GPIO0")
 			(pinfunction "Pin_11_11")
 			(pintype "passive")
@@
 			(layers "*.Cu" "*.Mask")
 			(remove_unused_layers no)
-			(net "unconnected-(J2-Pin_12-Pad12)")
+			(net "/GPIO1")
 			(pinfunction "Pin_12_12")
 			(pintype "passive")
@@
 			(net "unconnected-(J2-Pin_13-Pad13)")
 			(pinfunction "Pin_13_13")
-			(pintype "passive")
+			(pintype "passive+no_connect")
 		)
 		(pad "14" thru_hole circle
@@
 			(net "unconnected-(J2-Pin_14-Pad14)")
 			(pinfunction "Pin_14_14")
-			(pintype "passive")
+			(pintype "passive+no_connect")
 		)
 		(pad "15" thru_hole circle
@@
 			(net "unconnected-(J2-Pin_16-Pad16)")
 			(pinfunction "Pin_16_16")
-			(pintype "passive")
+			(pintype "passive+no_connect")
 		)
 		(pad "17" thru_hole circle
@@
 			(layers "*.Cu" "*.Mask")
 			(remove_unused_layers no)
-			(net "unconnected-(J2-Pin_21-Pad21)")
+			(net "+3.3V")
 			(pinfunction "Pin_21_21")
 			(pintype "passive")
@@
 			(layers "*.Cu" "*.Mask")
 			(remove_unused_layers no)
-			(net "unconnected-(J2-Pin_22-Pad22)")
+			(net "+3.3V")
 			(pinfunction "Pin_22_22")
 			(pintype "passive")
@@
 			(layers "*.Cu" "*.Mask")
 			(remove_unused_layers no)
-			(net "unconnected-(J2-Pin_23-Pad23)")
+			(net "GND")
 			(pinfunction "Pin_23_23")
 			(pintype "passive")
@@
 			(layers "*.Cu" "*.Mask")
 			(remove_unused_layers no)
-			(net "unconnected-(J2-Pin_24-Pad24)")
+			(net "GND")
 			(pinfunction "Pin_24_24")
 			(pintype "passive")
@@
 			(layers "*.Cu" "*.Mask")
 			(remove_unused_layers no)
-			(net "unconnected-(J2-Pin_37-Pad37)")
+			(net "+3.3V")
 			(pinfunction "Pin_37_37")
 			(pintype "passive")
@@
 			(layers "*.Cu" "*.Mask")
 			(remove_unused_layers no)
-			(net "unconnected-(J2-Pin_38-Pad38)")
+			(net "+3.3V")
 			(pinfunction "Pin_38_38")
 			(pintype "passive")
@@
 			(layers "*.Cu" "*.Mask")
 			(remove_unused_layers no)
-			(net "unconnected-(J2-Pin_39-Pad39)")
+			(net "GND")
 			(pinfunction "Pin_39_39")
 			(pintype "passive")
@@
 			(layers "*.Cu" "*.Mask")
 			(remove_unused_layers no)
-			(net "unconnected-(J2-Pin_40-Pad40)")
+			(net "GND")
 			(pinfunction "Pin_40_40")
 			(pintype "passive")
